Commit message: performance scripts from Europe, The White King film, and US travels

File: sophia/description.urdf (robot description, URDF)
Before this commit: robot han, 12 links, 11 joints
Joints:
- joint blender_joint: origin xyz=0 0 0.62 rpy=0 0.15 0 -> xyz=0 0 0.62 rpy=0 0 0
- joint body_camera: origin xyz=0.15 0 0.35 rpy=0 0 0 -> xyz=0.15 0 0.35 rpy=0 -0.3 0
